File: vine_badge.brd (EAGLE design)
At the start: 99.3 x 99.4 mm, 44 parts

Commit message: final checking phase
Parts:
- removed S1: (no value), SparkFun-Switches:SWITCH_DPDT_SMD_AYZ0202
- added D1: MBRA340T3, diode:SMA
- added ON/OFF: ON/OFF, VineBadge:SMT_DPDT
- added R7: 1k, resistor:R0603
- moved LED27 2.20 mm to (37.4, 88.9)
- turned S2 to 140 degrees
Connections:
- net N$10 renamed TPIDATA
- net N$8 renamed TPICLK
- removed net N$12: JP1.1, U$1.13
- new net N$20: D1.A, ON/OFF.P$1
- new net RESET: JP1.1, R7.2, U$1.13
- net +3V3: now also D1.C, R7.1; no longer S1.3
- net N$19: now also ON/OFF.P$2; no longer S1.2
Routing:
- net RESET: track 0.00 -> 22.0 mm, vias 0 -> 2
- net N$12: track 20.6 -> 0.00 mm, vias 1 -> 0
- net N$20: track 0.00 -> 9.69 mm
- net +3V3: track 103.8 -> 110.0 mm
- net N$6: track 177.5 -> 178.5 mm
- net TPICLK: track 18.0 -> 17.1 mm
- net N$2: vias 11 -> 10
Other:
- outline, holes or cut-outs redrawn

Commit message: small improvements
Routing:
- net N$1: track 134.4 -> 139.4 mm
- net N$2: track 179.8 -> 182.9 mm
- net +3V3: track 110.0 -> 112.7 mm
- net N$5: track 240.9 -> 243.1 mm
- net N$4: track 149.7 -> 150.9 mm
- net N$3: track 107.1 -> 107.8 mm

Commit message: added a wire I forgot about
Connections:
- removed net N$9: LED13.C, LED14.A
- net N$1: now also LED13.C, LED14.A
Routing:
- net N$1: track 139.4 -> 208.1 mm, vias 8 -> 10
- net N$9: track 12.3 -> 0.00 mm, vias 2 -> 0
Changed lines of the file:
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@@
 <layer number="14" name="Route14" color="22" fill="1" visible="no" active="no"/>
 <layer number="15" name="Route15" color="23" fill="1" visible="no" active="no"/>
-<layer number="16" name="Bottom" color="1" fill="1" visible="no" active="yes"/>
+<layer number="16" name="Bottom" color="1" fill="1" visible="yes" active="yes"/>
 <layer number="17" name="Pads" color="2" fill="1" visible="yes" active="yes"/>
 <layer number="18" name="Vias" color="2" fill="1" visible="yes" active="yes"/>
@@
 <layer number="20" name="Dimension" color="24" fill="1" visible="yes" active="yes"/>
 <layer number="21" name="tPlace" color="7" fill="1" visible="yes" active="yes"/>
-<layer number="22" name="bPlace" color="7" fill="1" visible="no" active="yes"/>
+<layer number="22" name="bPlace" color="7" fill="1" visible="yes" active="yes"/>
 <layer number="23" name="tOrigins" color="15" fill="1" visible="yes" active="yes"/>
-<layer number="24" name="bOrigins" color="15" fill="1" visible="no" active="yes"/>
+<layer number="24" name="bOrigins" color="15" fill="1" visible="yes" active="yes"/>
 <layer number="25" name="tNames" color="7" fill="1" visible="yes" active="yes"/>
-<layer number="26" name="bNames" color="7" fill="1" visible="no" active="yes"/>
+<layer number="26" name="bNames" color="7" fill="1" visible="yes" active="yes"/>
 <layer number="27" name="tValues" color="7" fill="1" visible="no" active="yes"/>
 <layer number="28" name="bValues" color="7" fill="1" visible="no" active="yes"/>
@@
 <layer number="38" name="bTest" color="7" fill="1" visible="no" active="yes"/>
 <layer number="39" name="tKeepout" color="4" fill="11" visible="yes" active="yes"/>
-<layer number="40" name="bKeepout" color="1" fill="11" visible="no" active="yes"/>
+<layer number="40" name="bKeepout" color="1" fill="11" visible="yes" active="yes"/>
 <layer number="41" name="tRestrict" color="4" fill="10" visible="yes" active="yes"/>
-<layer number="42" name="bRestrict" color="1" fill="10" visible="no" active="yes"/>
+<layer number="42" name="bRestrict" color="1" fill="10" visible="yes" active="yes"/>
 <layer number="43" name="vRestrict" color="2" fill="10" visible="no" active="yes"/>
 <layer number="44" name="Drills" color="7" fill="1" visible="no" active="yes"/>
@@
 <layer number="50" name="dxf" color="7" fill="1" visible="no" active="no"/>
 <layer number="51" name="tDocu" color="7" fill="1" visible="yes" active="yes"/>
-<layer number="52" name="bDocu" color="7" fill="1" visible="no" active="yes"/>
+<layer number="52" name="bDocu" color="7" fill="1" visible="yes" active="yes"/>
 <layer number="53" name="tGND_GNDA" color="7" fill="9" visible="no" active="no"/>
 <layer number="54" name="bGND_GNDA" color="1" fill="9" visible="no" active="no"/>
@@
 <wire x1="53.1622" y1="83.13434375" x2="52.84113125" y2="82.813275" width="0.2032" layer="1"/>
 <wire x1="52.84113125" y1="82.813275" x2="52.37585" y2="82.813275" width="0.2032" layer="1"/>
-</signal>
-<signal name="N$9">
 <contactref element="LED13" pad="C"/>
 <contactref element="LED14" pad="A"/>
@@
 <wire x1="39.170190625" y1="29.30729375" x2="39.162809375" y2="29.292965625" width="0.2032" layer="16"/>
 <wire x1="39.162809375" y1="29.292965625" x2="37.736246875" y2="28.661040625" width="0.2032" layer="16"/>
+<wire x1="63.754" y1="72.683" x2="63.754" y2="52.017425" width="0.2032" layer="1"/>
+<wire x1="40.25025625" y1="32.94100625" x2="39.8501625" y2="32.5409125" width="0.2032" layer="1"/>
+<wire x1="39.8501625" y1="32.5409125" x2="39.8501625" y2="31.9750875" width="0.2032" layer="1"/>
+<wire x1="39.8501625" y1="31.9750875" x2="40.25025625" y2="31.57499375" width="0.2032" layer="1"/>
+<wire x1="41.7165" y1="31.57499375" x2="42.514034375" y2="30.777459375" width="0.2032" layer="1"/>
+<wire x1="40.25025625" y1="31.57499375" x2="41.7165" y2="31.57499375" width="0.2032" layer="1"/>
+<wire x1="63.754" y1="52.017425" x2="44.67758125" y2="32.94100625" width="0.2032" layer="1"/>
+<wire x1="44.67758125" y1="32.94100625" x2="40.25025625" y2="32.94100625" width="0.2032" layer="1"/>
 </signal>
 <signal name="N$5">

Commit message: sent for manufacturing
Parts:
- D1: value MBRA340T3 -> BAT60J; device diode:SMA -> diode:SOD323_ST
Connections:
- net N$19: now also ON/OFF.P$5
- net N$20: now also ON/OFF.P$6
Routing:
- net N$20: track 9.69 -> 14.9 mm
- net N$19: track 36.1 -> 41.2 mm
- net N$9: track 0.00 -> 0.79 mm
- net N$10: track 0.00 -> 0.79 mm
- net N$8: track 0.00 -> 0.76 mm
- net N$21: track 0.00 -> 0.76 mm
- net N$12: track 0.00 -> 0.76 mm
Changed lines of the file:
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@@
 <grid distance="1" unitdist="mil" unit="mil" style="lines" multiple="1" display="yes" altdistance="5" altunitdist="mil" altunit="mil"/>
 <layers>
-<layer number="1" name="Top" color="12" fill="1" visible="yes" active="yes"/>
+<layer number="1" name="Top" color="12" fill="1" visible="no" active="yes"/>
 <layer number="2" name="Route2" color="16" fill="1" visible="no" active="no"/>
 <layer number="3" name="Route3" color="17" fill="1" visible="no" active="no"/>
@@
 <layer number="19" name="Unrouted" color="6" fill="1" visible="yes" active="yes"/>
 <layer number="20" name="Dimension" color="24" fill="1" visible="yes" active="yes"/>
-<layer number="21" name="tPlace" color="7" fill="1" visible="yes" active="yes"/>
+<layer number="21" name="tPlace" color="7" fill="1" visible="no" active="yes"/>
 <layer number="22" name="bPlace" color="7" fill="1" visible="yes" active="yes"/>
-<layer number="23" name="tOrigins" color="15" fill="1" visible="yes" active="yes"/>
+<layer number="23" name="tOrigins" color="15" fill="1" visible="no" active="yes"/>
 <layer number="24" name="bOrigins" color="15" fill="1" visible="yes" active="yes"/>
-<layer number="25" name="tNames" color="7" fill="1" visible="yes" active="yes"/>
+<layer number="25" name="tNames" color="7" fill="1" visible="no" active="yes"/>
 <layer number="26" name="bNames" color="7" fill="1" visible="yes" active="yes"/>
 <layer number="27" name="tValues" color="7" fill="1" visible="no" active="yes"/>
-<layer number="28" name="bValues" color="7" fill="1" visible="no" active="yes"/>
+<layer number="28" name="bValues" color="7" fill="1" visible="yes" active="yes"/>
 <layer number="29" name="tStop" color="7" fill="3" visible="no" active="yes"/>
-<layer number="30" name="bStop" color="7" fill="6" visible="no" active="yes"/>
+<layer number="30" name="bStop" color="7" fill="6" visible="yes" active="yes"/>
 <layer number="31" name="tCream" color="7" fill="4" visible="no" active="yes"/>
 <layer number="32" name="bCream" color="7" fill="5" visible="no" active="yes"/>
@@
 <layer number="37" name="tTest" color="7" fill="1" visible="no" active="yes"/>
 <layer number="38" name="bTest" color="7" fill="1" visible="no" active="yes"/>
-<layer number="39" name="tKeepout" color="4" fill="11" visible="yes" active="yes"/>
+<layer number="39" name="tKeepout" color="4" fill="11" visible="no" active="yes"/>
 <layer number="40" name="bKeepout" color="1" fill="11" visible="yes" active="yes"/>
-<layer number="41" name="tRestrict" color="4" fill="10" visible="yes" active="yes"/>
+<layer number="41" name="tRestrict" color="4" fill="10" visible="no" active="yes"/>
 <layer number="42" name="bRestrict" color="1" fill="10" visible="yes" active="yes"/>
-<layer number="43" name="vRestrict" color="2" fill="10" visible="no" active="yes"/>
+<layer number="43" name="vRestrict" color="2" fill="10" visible="yes" active="yes"/>
 <layer number="44" name="Drills" color="7" fill="1" visible="no" active="yes"/>
 <layer number="45" name="Holes" color="7" fill="1" visible="no" active="yes"/>
@@
 <layer number="49" name="Reference" color="7" fill="1" visible="no" active="yes"/>
 <layer number="50" name="dxf" color="7" fill="1" visible="no" active="no"/>
-<layer number="51" name="tDocu" color="7" fill="1" visible="yes" active="yes"/>
+<layer number="51" name="tDocu" color="7" fill="1" visible="no" active="yes"/>
 <layer number="52" name="bDocu" color="7" fill="1" visible="yes" active="yes"/>
 <layer number="53" name="tGND_GNDA" color="7" fill="9" visible="no" active="no"/>
@@
 <attribute name="VALUE" x="78.994378125" y="94.740403125" size="1.27" layer="27" rot="R153.5"/>
 </element>
-<element name="D1" library="diode" library_urn="urn:adsk.eagle:library:210" package="SMA" package3d_urn="urn:adsk.eagle:package:43460/3" value="MBRA340T3" x="39.4716" y="43.2308" smashed="yes" rot="MR0">
+<element name="D1" library="diode" library_urn="urn:adsk.eagle:library:210" package="SOD323_ST" package3d_urn="urn:adsk.eagle:package:43461/1" value="BAT60J" x="39.4716" y="43.2308" smashed="yes" rot="MR0">
 <attribute name="NAME" x="40.342" y="45.4848" size="1.27" layer="26" font="vector" ratio="20" rot="MR0"/>
 </element>
@@
 <wire x1="62.23" y1="37.592" x2="58.166" y2="35.814" width="0.4064" layer="1"/>
 <contactref element="D1" pad="C"/>
-<wire x1="41.4716" y1="43.2308" x2="40.533165625" y2="42.292365625" width="0.4064" layer="16"/>
+<wire x1="40.7216" y1="43.2308" x2="40.533165625" y2="42.292365625" width="0.4064" layer="16"/>
 <wire x1="40.533165625" y1="42.292365625" x2="40.533165625" y2="32.258" width="0.4064" layer="16"/>
 <via x="40.533165625" y="32.258" extent="1-16" drill="0.35"/>
@@
 <wire x1="36.69085625" y1="57.84978125" x2="33.032428125" y2="61.508209375" width="0.2032" layer="16"/>
 <wire x1="42.384496875" y1="57.081440625" x2="41.61615625" y2="57.84978125" width="0.2032" layer="16"/>
-<wire x1="57.404" y1="77.724" x2="57.57" y2="77.724" width="0.2032" layer="16"/>
 <wire x1="30.90895625" y1="76.088709375" x2="32.258128125" y2="77.43788125" width="0.2032" layer="16"/>
 <wire x1="13.708346875" y1="56.597584375" x2="28.121803125" y2="56.597584375" width="0.2032" layer="1"/>
 <wire x1="28.121803125" y1="56.597584375" x2="33.032428125" y2="61.508209375" width="0.2032" layer="1"/>
-<wire x1="57.11788125" y1="77.43788125" x2="57.404" y2="77.724" width="0.2032" layer="16"/>
 <wire x1="32.258128125" y1="77.43788125" x2="57.11788125" y2="77.43788125" width="0.2032" layer="16"/>
 <wire x1="30.52724375" y1="28.01975625" x2="31.41624375" y2="28.01975625" width="0.2032" layer="16"/>
@@
 <wire x1="1.733878125" y1="40.4999625" x2="1.579103125" y2="39.468128125" width="0.2032" layer="1"/>
 <wire x1="1.579103125" y1="39.468128125" x2="1.579103125" y2="37.239425" width="0.2032" layer="1"/>
+<wire x1="57.57" y1="77.724" x2="57.11788125" y2="77.43788125" width="0.2032" layer="16"/>
 </signal>
 <signal name="N$3">
@@
 <wire x1="27.892821875" y1="87.575578125" x2="30.336325" y2="87.446553125" width="0.2032" layer="16"/>
 <wire x1="31.4347" y1="87.446553125" x2="30.336325" y2="87.446553125" width="0.2032" layer="16"/>
-<wire x1="32.139059375" y1="88.1509125" x2="32.128571875" y2="88.140425" width="0.2032" layer="16"/>
 <wire x1="32.128571875" y1="88.140425" x2="31.4347" y2="87.446553125" width="0.2032" layer="16"/>
 <wire x1="32.50248125" y1="88.304003125" x2="32.2961625" y2="88.21374375" width="0.2032" layer="16"/>
@@
 <contactref element="U$2" pad="P$2"/>
 <wire x1="7.88775625" y1="36.230946875" x2="17.7007875" y2="44.465053125" width="1.016" layer="16"/>
-<wire x1="17.7007875" y1="44.465053125" x2="29.845" y2="32.320840625" width="0.4064" layer="16"/>
+<wire x1="17.7007875" y1="44.465053125" x2="29.591" y2="32.574840625" width="0.4064" layer="16"/>
 <contactref element="ON/OFF" pad="P$2"/>
-<wire x1="29.845" y1="32.320840625" x2="35.635390625" y2="32.320840625" width="0.4064" layer="16"/>
-<wire x1="35.635390625" y1="32.320840625" x2="35.888165625" y2="32.068065625" width="0.4064" layer="16"/>
+<wire x1="29.591" y1="32.574840625" x2="34.972390625" y2="32.574840625" width="0.4064" layer="16"/>
+<wire x1="34.972390625" y1="32.574840625" x2="35.695328125" y2="32.297878125" width="0.4064" layer="16"/>
+<contactref element="ON/OFF" pad="P$5"/>
+<wire x1="32.224275" y1="36.43451875" x2="35.695328125" y2="32.297878125" width="0.4064" layer="16"/>
 </signal>
 <signal name="N$18">
@@
 <contactref element="D1" pad="A"/>
 <contactref element="ON/OFF" pad="P$1"/>
-<wire x1="37.803275" y1="42.899125" x2="37.4716" y2="43.2308" width="0.4064" layer="16"/>
-<wire x1="37.803275" y1="33.675034375" x2="37.803275" y2="42.899125" width="0.4064" layer="16"/>
+<wire x1="37.803275" y1="42.899125" x2="38.2216" y2="43.2308" width="0.4064" layer="16"/>
+<wire x1="37.610440625" y1="33.904846875" x2="37.803275" y2="42.899125" width="0.4064" layer="16"/>
+<contactref element="ON/OFF" pad="P$6"/>
+<wire x1="34.1393875" y1="38.0414875" x2="37.610440625" y2="33.904846875" width="0.4064" layer="16"/>
+</signal>
+<signal name="N$8">
+<wire x1="58.8518" y1="79.8576" x2="58.0898" y2="79.8576" width="0.2032" layer="16"/>
+</signal>
+<signal name="N$9">
+<wire x1="58.0136" y1="77.724" x2="58.801" y2="77.724" width="0.2032" layer="16"/>
+</signal>
+<signal name="N$10">
+<wire x1="58.0136" y1="75.6666" x2="58.801" y2="75.6666" width="0.2032" layer="16"/>
+</signal>
+<signal name="N$12">
+<wire x1="58.0136" y1="73.6346" x2="58.7756" y2="73.6346" width="0.2032" layer="16"/>
+</signal>
+<signal name="N$21">
+<wire x1="58.0136" y1="81.915" x2="58.7756" y2="81.915" width="0.2032" layer="16"/>
 </signal>
 </signals>
