File: vine_badge.brd (EAGLE design)
At the start: 99.3 x 99.4 mm, 46 parts

Commit message: small fixes for pcb run 2
Parts:
- D1: value BAT60J -> (none); device diode:SOD323_ST -> diode:SOD523
Routing:
- net N$22: track 0.00 -> 1.71 mm
- net N$18: track 5.92 -> 7.23 mm
- net N$16: track 3.55 -> 4.19 mm
- net N$13: track 3.48 -> 4.11 mm
- net N$20: track 14.9 -> 15.5 mm
Changed lines of the file:
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@@
 <attribute name="VALUE" x="78.994378125" y="94.740403125" size="1.27" layer="27" rot="R153.5"/>
 </element>
-<element name="D1" library="diode" library_urn="urn:adsk.eagle:library:210" package="SOD323_ST" package3d_urn="urn:adsk.eagle:package:43461/1" value="BAT60J" x="39.4716" y="43.2308" smashed="yes" rot="MR0">
+<element name="D1" library="diode" library_urn="urn:adsk.eagle:library:210" package="SOD523" package3d_urn="urn:adsk.eagle:package:43410/1" value="" x="39.4716" y="43.2308" smashed="yes" rot="MR0">
 <attribute name="NAME" x="40.342" y="45.4848" size="1.27" layer="26" font="vector" ratio="20" rot="MR0"/>
 </element>
@@
 <wire x1="62.723" y1="88.138" x2="62.723" y2="83.3098" width="0.4064" layer="16"/>
 <wire x1="62.723" y1="83.3098" x2="62.7294" y2="83.3034" width="0.4064" layer="16"/>
-<wire x1="63.7894" y1="79.995" x2="63.7894" y2="82.2434" width="0.3048" layer="16"/>
+<wire x1="63.7894" y1="79.845" x2="63.7894" y2="82.2434" width="0.3048" layer="16"/>
 <wire x1="63.7894" y1="82.2434" x2="63.881" y2="82.335" width="0.3048" layer="16"/>
 <wire x1="40.533165625" y1="32.258" x2="44.196" y2="32.258" width="0.4064" layer="1"/>
@@
 <wire x1="62.23" y1="37.592" x2="58.166" y2="35.814" width="0.4064" layer="1"/>
 <contactref element="D1" pad="C"/>
-<wire x1="40.7216" y1="43.2308" x2="40.533165625" y2="42.292365625" width="0.4064" layer="16"/>
-<wire x1="40.533165625" y1="42.292365625" x2="40.533165625" y2="32.258" width="0.4064" layer="16"/>
 <via x="40.533165625" y="32.258" extent="1-16" drill="0.35"/>
 <contactref element="R7" pad="1"/>
@@
 <wire x1="71.23818125" y1="46.406403125" x2="71.315290625" y2="46.4835125" width="0.4064" layer="1"/>
 <wire x1="71.315290625" y1="46.4835125" x2="71.320153125" y2="46.4835125" width="0.4064" layer="1"/>
+<wire x1="40.0716" y1="43.2308" x2="40.533165625" y2="42.769234375" width="0.4064" layer="16"/>
+<wire x1="40.533165625" y1="42.769234375" x2="40.533165625" y2="32.258" width="0.4064" layer="16"/>
 </signal>
 <signal name="GND">
@@
 <signal name="TPICLK">
 <contactref element="U$1" pad="11"/>
-<wire x1="65.0394" y1="79.245" x2="66.421" y2="80.01" width="0.2032" layer="16"/>
+<wire x1="64.8894" y1="79.245" x2="64.988171875" y2="79.294334375" width="0.2032" layer="16"/>
 <via x="66.421" y="80.01" extent="1-16" drill="0.35"/>
 <contactref element="JP1" pad="3"/>
@@
 <wire x1="67.8165375" y1="83.53915625" x2="71.32795" y2="92.6627625" width="0.2032" layer="1"/>
 <wire x1="66.840209375" y1="81.19826875" x2="67.8165375" y2="83.53915625" width="0.2032" layer="1"/>
+<wire x1="64.988171875" y1="79.294334375" x2="65.705334375" y2="79.294334375" width="0.2032" layer="16"/>
+<wire x1="65.705334375" y1="79.294334375" x2="66.421" y2="80.01" width="0.2032" layer="16"/>
 </signal>
 <signal name="TPIDATA">
 <contactref element="U$1" pad="12"/>
 <via x="67.3806" y="79.883" extent="1-16" drill="0.35"/>
-<wire x1="65.0394" y1="78.745" x2="65.3846" y2="78.7902" width="0.2032" layer="16"/>
+<wire x1="64.8894" y1="78.745" x2="65.3846" y2="78.7902" width="0.2032" layer="16"/>
 <wire x1="67.2599125" y1="79.883" x2="67.3806" y2="79.883" width="0.2032" layer="16"/>
 <wire x1="65.3846" y1="78.7902" x2="66.1671125" y2="78.7902" width="0.2032" layer="16"/>
@@
 <contactref element="U$1" pad="13"/>
 <via x="68.3402" y="79.883" extent="1-16" drill="0.35"/>
-<wire x1="65.0394" y1="78.245" x2="65.3846" y2="78.2902" width="0.2032" layer="16"/>
+<wire x1="64.8894" y1="78.245" x2="65.3846" y2="78.2902" width="0.2032" layer="16"/>
 <wire x1="68.0636" y1="79.6000875" x2="68.0636" y2="79.6064" width="0.2032" layer="16"/>
 <wire x1="68.0636" y1="79.6064" x2="68.3402" y2="79.883" width="0.2032" layer="16"/>
@@
 <contactref element="U$1" pad="1"/>
 <contactref element="R5" pad="1"/>
-<wire x1="61.5394" y1="77.245" x2="60.866" y2="76.8716" width="0.2032" layer="16"/>
 <wire x1="59.27" y1="74.21095" x2="59.27" y2="73.66" width="0.2032" layer="16"/>
-<wire x1="60.866" y1="76.8716" x2="60.866" y2="75.80695" width="0.2032" layer="16"/>
+<wire x1="60.866" y1="76.8716" x2="60.866" y2="76.4794" width="0.2032" layer="16"/>
+<wire x1="60.866" y1="75.80695" x2="60.866" y2="76.4794" width="0.2032" layer="16"/>
 <wire x1="60.866" y1="75.80695" x2="59.27" y2="74.21095" width="0.2032" layer="16"/>
+<wire x1="61.6894" y1="77.245" x2="61.4172" y2="77.245" width="0.2032" layer="16"/>
+<wire x1="61.4172" y1="77.245" x2="61.2394" y2="77.245" width="0.2032" layer="16"/>
+<wire x1="61.2394" y1="77.245" x2="60.866" y2="76.8716" width="0.2032" layer="16"/>
+<wire x1="60.866" y1="76.4794" x2="60.866" y2="76.4794" width="0.2032" layer="16"/>
 </signal>
 <signal name="N$13">
 <contactref element="U$1" pad="2"/>
 <contactref element="R4" pad="1"/>
-<wire x1="59.27" y1="75.7756" x2="59.27" y2="75.692" width="0.2032" layer="16"/>
-<wire x1="61.5394" y1="77.745" x2="61.1942" y2="77.6998" width="0.2032" layer="16"/>
-<wire x1="61.1942" y1="77.6998" x2="60.63815" y2="77.6998" width="0.2032" layer="16"/>
-<wire x1="60.63815" y1="77.6998" x2="60.4596" y2="77.52125" width="0.2032" layer="16"/>
-<wire x1="60.4596" y1="76.9652" x2="59.27" y2="75.7756" width="0.2032" layer="16"/>
-<wire x1="60.4596" y1="77.52125" x2="60.4596" y2="76.9652" width="0.2032" layer="16"/>
+<wire x1="59.27" y1="75.8503375" x2="59.27" y2="75.692" width="0.2032" layer="16"/>
+<wire x1="61.6894" y1="77.745" x2="60.9556" y2="77.745" width="0.2032" layer="16"/>
+<wire x1="60.3758" y1="77.1652" x2="60.3758" y2="75.9968" width="0.2032" layer="16"/>
+<wire x1="60.3758" y1="75.9968" x2="60.071" y2="75.692" width="0.2032" layer="16"/>
+<wire x1="60.071" y1="75.692" x2="59.27" y2="75.692" width="0.2032" layer="16"/>
+<wire x1="60.9556" y1="77.745" x2="60.3758" y2="77.1652" width="0.2032" layer="16"/>
 </signal>
 <signal name="N$14">
 <contactref element="U$1" pad="3"/>
 <contactref element="R3" pad="1"/>
-<wire x1="61.5394" y1="78.245" x2="59.791" y2="78.245" width="0.2032" layer="16"/>
+<wire x1="61.6894" y1="78.245" x2="59.791" y2="78.245" width="0.2032" layer="16"/>
 <wire x1="59.791" y1="78.245" x2="59.27" y2="77.724" width="0.2032" layer="16"/>
 </signal>
@@
 <contactref element="U$1" pad="4"/>
 <contactref element="R2" pad="1"/>
-<wire x1="61.5394" y1="78.745" x2="60.408" y2="78.745" width="0.2032" layer="16"/>
+<wire x1="61.6894" y1="78.745" x2="60.408" y2="78.745" width="0.2032" layer="16"/>
 <wire x1="60.408" y1="78.745" x2="59.27" y2="79.883" width="0.2032" layer="16"/>
 </signal>
@@
 <contactref element="U$1" pad="5"/>
 <contactref element="R1" pad="1"/>
-<wire x1="59.27" y1="81.915" x2="61.2394" y2="79.9456" width="0.2032" layer="16"/>
-<wire x1="61.2394" y1="79.9456" x2="61.5394" y2="79.245" width="0.2032" layer="16"/>
+<wire x1="59.27" y1="81.915" x2="59.4038" y2="81.7812" width="0.2032" layer="16"/>
+<wire x1="61.6894" y1="79.245" x2="60.8106" y2="79.245" width="0.2032" layer="16"/>
+<wire x1="60.0748" y1="79.9808" x2="60.0748" y2="80.55925" width="0.2032" layer="16"/>
+<wire x1="59.4038" y1="81.23025" x2="59.4038" y2="81.7812" width="0.2032" layer="16"/>
+<wire x1="60.0748" y1="80.55925" x2="59.4038" y2="81.23025" width="0.2032" layer="16"/>
+<wire x1="60.8106" y1="79.245" x2="60.0748" y2="79.9808" width="0.2032" layer="16"/>
 </signal>
 <signal name="N$17">
 <contactref element="R6" pad="1"/>
 <contactref element="U$1" pad="17"/>
-<wire x1="63.7894" y1="76.495" x2="63.754" y2="76.1596" width="0.2032" layer="16"/>
+<wire x1="63.7894" y1="76.645" x2="63.754" y2="76.1596" width="0.2032" layer="16"/>
 <wire x1="63.754" y1="76.1596" x2="63.754" y2="74.383" width="0.2032" layer="16"/>
 </signal>
@@
 <contactref element="U$1" pad="16"/>
 <contactref element="S2" pad="1"/>
-<wire x1="64.2894" y1="76.495" x2="67.289234375" y2="76.195" width="0.2032" layer="16"/>
-<wire x1="67.289234375" y1="76.195" x2="69.4689625" y2="78.11221875" width="0.2032" layer="16"/>
+<wire x1="64.2894" y1="76.645" x2="64.2894" y2="75.9694" width="0.2032" layer="16"/>
+<wire x1="64.2894" y1="75.9694" x2="64.8716" y2="75.3872" width="0.2032" layer="16"/>
+<wire x1="64.8716" y1="75.3872" x2="66.496528125" y2="75.3872" width="0.2032" layer="16"/>
+<wire x1="69.221546875" y1="78.11221875" x2="69.4689625" y2="78.11221875" width="0.2032" layer="16"/>
+<wire x1="66.496528125" y1="75.3872" x2="69.221546875" y2="78.11221875" width="0.2032" layer="16"/>
 </signal>
 <signal name="SHADOW">
@@
 <contactref element="D1" pad="A"/>
 <contactref element="ON/OFF" pad="P$1"/>
-<wire x1="37.803275" y1="42.899125" x2="38.2216" y2="43.2308" width="0.4064" layer="16"/>
-<wire x1="37.610440625" y1="33.904846875" x2="37.803275" y2="42.899125" width="0.4064" layer="16"/>
+<wire x1="37.803275" y1="42.899125" x2="37.610440625" y2="33.904846875" width="0.4064" layer="16"/>
 <contactref element="ON/OFF" pad="P$6"/>
 <wire x1="34.1393875" y1="38.0414875" x2="37.610440625" y2="33.904846875" width="0.4064" layer="16"/>
+<wire x1="38.7716" y1="43.2308" x2="38.13495" y2="43.2308" width="0.4064" layer="16"/>
+<wire x1="38.13495" y1="43.2308" x2="37.803275" y2="42.899125" width="0.4064" layer="16"/>
 </signal>
 <signal name="N$8">
@@
 <wire x1="58.0136" y1="81.915" x2="58.7756" y2="81.915" width="0.2032" layer="16"/>
 </signal>
+<signal name="N$22">
+<wire x1="63.7286" y1="74.3712" x2="63.7286" y2="72.6948" width="0.2032" layer="16"/>
+<wire x1="63.7286" y1="72.6948" x2="63.754" y2="72.6694" width="0.2032" layer="16"/>
+</signal>
 </signals>

Commit message: moved to v 1.1
Parts:
- added FRAME1: FRAME-LETTER, SparkFun-Aesthetics:CREATIVE_COMMONS
- added FUSE: 1206_FUSE, VineBadge:R1206
- added JP2: JUMPER-SMT_2_NC_TRACE_NO-SILK, SparkFun-Jumpers:SMT-JUMPER_2_NC_TRACE_NO-SILK
- added JP3: JUMPER-SMT_2_NO_NO-SILK, SparkFun-Jumpers:SMT-JUMPER_2_NO_NO-SILK
- added LOGO1: OSHW-LOGOS-COPPER, SparkFun-Aesthetics:OSHW-LOGO-S_COPPER
- added U$4: SI2312, VineBadge:SOT23
- moved D1 19.3 mm to (24.9, 30.6)
Connections:
- new net MODE: S2.1, U$1.14
- new net N$23: D1.C, JP2.2, ON/OFF.P$2, ON/OFF.P$5
- net +3V3: now also ON/OFF.P$1, ON/OFF.P$6, U$4.1; no longer D1.C
- net GND: now also JP3.2, U$4.2; no longer U$3.P$3, U$3.P$4
- net N$18: now also FUSE.1, U$2.P$1, U$2.P$2; no longer S2.1, U$1.16
- net N$19: now also JP3.1, U$3.P$3, U$3.P$4, U$4.3; no longer ON/OFF.P$2, ON/OFF.P$5, U$2.P$1, U$2.P$2
- net N$20: now also FUSE.2, JP2.1; no longer ON/OFF.P$1, ON/OFF.P$6
Routing:
- net N$19: track 41.2 -> 20.6 mm
- net N$23: track 0.00 -> 19.1 mm
- net N$18: track 7.23 -> 26.0 mm
- net +3V3: track 113.0 -> 131.4 mm, vias 2 -> 4
- net N$20: track 15.5 -> 7.03 mm
- net MODE: track 0.00 -> 4.73 mm
- net GND: track 12.8 -> 9.96 mm
- net N$1: track 208.1 -> 209.8 mm
- net N$22: track 1.71 -> 0.04 mm
- added copper zone on layer 16, net YAHAHA
Other:
- board text added: "+"
- board text added: "CC BY-SA 4.0"
- board text added: "TMG 2019"
- board text added: "Yahaha!"
