File: vine_badge.sch (EAGLE design)
At the start: 46 parts

Commit message: small fixes for pcb run 2
Parts:
- D1: value BAT60J -> (none); device diode:BAT60J -> diode:DIODE-SOD523
Changed lines of the file:
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@@
 <part name="S2" library="SparkFun-Switches" library_urn="urn:adsk.eagle:library:535" deviceset="MOMENTARY-SWITCH-SPST" device="-SMD-6.0X3.5MM" package3d_urn="urn:adsk.eagle:package:40165/1" value="MODE"/>
 <part name="JP1" library="pinhead" library_urn="urn:adsk.eagle:library:325" deviceset="PINHD-1X3" device="" package3d_urn="urn:adsk.eagle:package:22458/2"/>
-<part name="D1" library="diode" library_urn="urn:adsk.eagle:library:210" deviceset="BAT60J" device="" package3d_urn="urn:adsk.eagle:package:43461/1"/>
+<part name="D1" library="diode" library_urn="urn:adsk.eagle:library:210" deviceset="DIODE-" device="SOD523" package3d_urn="urn:adsk.eagle:package:43410/1"/>
 <part name="R7" library="resistor" library_urn="urn:adsk.eagle:library:348" deviceset="R-US_" device="R0603" package3d_urn="urn:adsk.eagle:package:23555/2" value="1k"/>
 <part name="+3V3" library="supply1" library_urn="urn:adsk.eagle:library:371" deviceset="+3V3" device=""/>

Commit message: moved to v 1.1
Parts:
- added FRAME1: FRAME-LETTER, SparkFun-Aesthetics:FRAME-LETTER
- added FUSE: 1206_FUSE, VineBadge:1206_FUSE
- added JP2: JUMPER-SMT_2_NC_TRACE_NO-SILK, SparkFun-Jumpers:JUMPER-SMT_2_NC_TRACE_NO-SILK
- added JP3: JUMPER-SMT_2_NO_NO-SILK, SparkFun-Jumpers:JUMPER-SMT_2_NO_NO-SILK
- added LOGO1: OSHW-LOGOS-COPPER, SparkFun-Aesthetics:OSHW-LOGOS-COPPER
- added U$4: SI2312, VineBadge:SI2312
Connections:
- new net MODE: S2.1, U$1G$2.PB2(CKOUT/OC0A/OC1B/MISO/INT0/PCINT10)
- new net N$23: D1.C, JP2.2, ON/OFF.P$2, ON/OFF.P$5
- net +3V3: now also ON/OFF.P$1, ON/OFF.P$6, U$4.G; no longer D1.C
- net GND: now also JP3.2, U$4.S; no longer U$3.NEG1
- net N$18: now also FUSE.1, U$2.POS1; no longer S2.1, U$1G$2.PA6(ADC6/PCINT6/!SS!)
- net N$19: now also JP3.1, U$3.NEG1, U$4.D; no longer ON/OFF.P$2, ON/OFF.P$5, U$2.POS1
- net N$20: now also FUSE.2, JP2.1; no longer ON/OFF.P$1, ON/OFF.P$6
Other:
- note added: "1.1"
- note added: "4/17/19"
- note added: "ATTiny20 MCU"
- note added: "Charlieplex LED Array"
- note added: "Grant Haack"
- note added: "Power Management"
- note added: "Vinesauce TMG Badge 2019"
- note added: "granthaack.com"
- moved on the sheet: C1, C2, D1, JP1, LED1, LED10, LED11, LED12, LED13, LED14, LED15, LED16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
